File: KiCad/DaisyDelayHardware.kicad_pcb (KiCad board)
At the start: 2 copper layers, 110.8 x 128.5 mm, 55 parts, among them J1 AUDIO_OUTPUT, J2 FEEDBACK_CV_INPUT, J3 DELAY_TIME_CV_INPUT, J4 EURO_PWR_2x8, J5 AUDIO_INPUT, SW1 SW_SPDT, U1 LM4040DBZ-10, U2 TL074, U4 MCP6002-xP

Commit message: update
Parts:
- removed HEAD1: PinHeader, Connector_PinHeader_2.54mm:PinHeader_1x20_P2.54mm_Vertical
- removed HEAD2: PinHeader_1x20_P2.54mm_Vertical, Connector_PinHeader_2.54mm:PinHeader_1x20_P2.54mm_Vertical
- removed REF** (x2): Eurorack_Panel_ScrewHole_Oval, Library:Eurorack_Panel_ScrewHole_Oval
- removed SOCK1: PinSocket, Connector_PinSocket_2.54mm:PinSocket_1x20_P2.54mm_Vertical
- removed SOCK1: PinSocket_1x20_P2.54mm_Vertical, Connector_PinSocket_2.54mm:PinSocket_1x20_P2.54mm_Vertical
- removed U4: MCP6002-xP, Package_DIP:DIP-8_W7.62mm
- added HEAD_L1: PinHeader, Connector_PinHeader_2.54mm:PinHeader_1x20_P2.54mm_Vertical, F.Cu at (207.0, 41.7)
- added HEAD_R1: PinHeader, Connector_PinHeader_2.54mm:PinHeader_1x20_P2.54mm_Vertical, F.Cu at (229.9, 41.7)
- added SOCK_L1: PinSocket, Connector_PinSocket_2.54mm:PinSocket_1x20_P2.54mm_Vertical, B.Cu at (189.2, 41.7)
- added SOCK_R1: PinSocket, Connector_PinSocket_2.54mm:PinSocket_1x20_P2.54mm_Vertical, B.Cu at (166.4, 41.7)
- added U3: MCP6002-xP, Package_DIP:DIP-8_W7.62mm, F.Cu at (219.6, 117.7)
- SW1: footprint Connector_Wire:SolderWire-0.5sqmm_1x02_P4.6mm_D0.9mm_OD2.1mm -> Library:SW_Slide-03_Wuerth-WS-SLTV_10x2.5x6.4_P2.54mm-SolderLugs
- moved R9 29.4 mm to (220.9, 79.8)
- moved R12 27.1 mm to (231.0, 95.6), turned to 180 degrees
- moved R6 23.4 mm to (218.3, 84.9)
- moved R10 20.4 mm to (223.4, 87.5)
- moved R11 20.1 mm to (225.9, 93.0), turned to 0 degrees
- moved C7 18.0 mm to (227.2, 110.3), turned to 0 degrees
- moved C8 15.2 mm to (229.5, 117.7), turned to -90 degrees
- moved R8 14.4 mm to (214.1, 96.1), turned to 180 degrees
- moved J1 14.0 mm to (184.8, 133.2)
- moved J5 14.0 mm to (170.8, 133.2)
- moved R4 13.4 mm to (217.3, 125.5), turned to 90 degrees
- moved R7 12.8 mm to (223.4, 84.9), turned to 90 degrees
- moved C6 9.97 mm to (231.5, 125.0), turned to 90 degrees
- moved R19 9.39 mm to (214.8, 125.5), turned to 90 degrees
- moved U1 8.46 mm to (228.5, 113.8)
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Connections:
- net +5V renamed H_+5V
- net -10V_REF renamed S_-10V_REF
- net 3V3_A renamed H_3V3_A
- net ADC_IN_0 renamed H_ADC_IN_0
- net ADC_IN_1 renamed H_ADC_IN_1
- net AUDIO_IN_L renamed H_AUDIO_IN_L
- net AUDIO_OUT_L renamed H_AUDIO_OUT_L
- net H6 renamed H_-10V_REF
- net H_GND renamed GND
- C11 pad 1: -12V -> Net-(C11-Pad1)
- C12 pad 2: +12V -> Net-(C12-Pad2)
- C13 pad 2: +12V -> Net-(C12-Pad2)
- C14 pad 1: -12V -> Net-(C11-Pad1)
- D1 pad 1: unconnected-(D1-K-Pad1) -> S_GND
- J4 pad 1: -12V -> Net-(C11-Pad1)
- J4 pad 10: +12V -> Net-(C12-Pad2)
- J4 pad 2: -12V -> Net-(C11-Pad1)
- J4 pad 9: +12V -> Net-(C12-Pad2)
- R19 pad 1: +12V -> Net-(C12-Pad2)
- SEED1 pad 12: H5 -> H_SWITCH_IN
- SW1 pad 2: S5 -> S_SWITCH_IN
Routing:
- net GND: track 0.00 -> 180.4 mm
- net H_+5V: track 0.00 -> 106.8 mm
- net S4: track 132.0 -> 32.2 mm
- net H_ADC_IN_1: track 0.00 -> 79.1 mm
- net S5: track 77.0 -> 0.00 mm
- net H_3V3_A: track 0.00 -> 73.9 mm, vias 0 -> 2
- net S_SWITCH_IN: track 0.00 -> 68.2 mm
- net H_ADC_IN_0: track 0.00 -> 63.5 mm, vias 0 -> 1
- net H4: track 0.00 -> 57.5 mm, vias 0 -> 1
- net H3: track 0.00 -> 56.7 mm
- net S1: track 111.9 -> 61.9 mm
- net H_-10V_REF: track 0.00 -> 48.1 mm, vias 0 -> 1
- net +12V: track 0.00 -> 45.3 mm
- net S2: track 97.1 -> 55.2 mm
- net H2: track 0.00 -> 33.6 mm
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Other:
- board size 110.8 x 128.5 mm -> 120.9 x 128.5 mm
- board text added: "AUDIO IN"
- board text added: "AUDIO OUT"
- board text added: "JLCJLCJLCJLC"
- board text added: "LED"
- board text added: "P1"
- board text added: "P1 CV"
- board text added: "P2"
- board text added: "P2 CV"
- board text added: "SEED FX"
- board text added: "SWITCH"
- board text added: "SynthLab"
