File: KiCad/DaisyDelayHardware.kicad_sch (KiCad schematic)
At the start: 51 parts, among them J1 AUDIO_OUTPUT, J2 FEEDBACK_CV_INPUT, J3 DELAY_TIME_CV_INPUT, J4 EURO_PWR_2x8, J5 AUDIO_INPUT, SW1 SW_SPDT, U1 LM4040DBZ-10, U2 TL074, U4 MCP6002-xP

Commit message: update
Parts:
- removed U4: MCP6002-xP, Package_DIP:DIP-8_W7.62mm, symbol Amplifier_Operational:MCP6002-xP
- added HEAD_R1: PinHeader, Connector_PinHeader_2.54mm:PinHeader_1x20_P2.54mm_Vertical, symbol Connector_Generic:Conn_01x20
- added SOCK_R1: PinSocket, Connector_PinSocket_2.54mm:PinSocket_1x20_P2.54mm_Vertical, symbol Connector_Generic:Conn_01x20
- added U3: MCP6002-xP, Package_DIP:DIP-8_W7.62mm, symbol Amplifier_Operational:MCP6002-xP
- R1, R10, R11, R12, R13, R14, R15, R16, R17, R18, R19, R2, R20, R3, R4, R5, R6, R7, R8, R9: footprint Resistor_THT:R_Axial_DIN0207_L6.3mm_D2.5mm_P10.16mm_Horizontal -> Resistor_THT:R_Axial_DIN0204_L3.6mm_D1.6mm_P5.08mm_Horizontal
- SW1: footprint Connector_Wire:SolderWire-0.5sqmm_1x02_P4.6mm_D0.9mm_OD2.1mm -> Library:SW_Slide-03_Wuerth-WS-SLTV_10x2.5x6.4_P2.54mm-SolderLugs
- renumbered HEAD1 to HEAD_L1, SOCK1 to SOCK_L1
Connections:
- net +12V: no longer C12.2, C13.2, J4.10 (+12V), J4.9 (+12V), R19.1
- net -12V: no longer C11.1, C14.1, J4.1 (-12V), J4.2 (-12V)
- net GND: now also HEAD_R1.18 (Pin_18), U3.3 (+), U3.4 (V-), U3.5 (+); no longer HEAD_L1.9 (Pin_9)
- net H1: now also HEAD_L1.17 (Pin_17); no longer HEAD_L1.1 (Pin_1)
- net H2: now also HEAD_L1.18 (Pin_18); no longer HEAD_L1.2 (Pin_2)
- net H3: now also HEAD_L1.19 (Pin_19), U3.2 (-); no longer HEAD_L1.3 (Pin_3)
- net H4: now also HEAD_L1.20 (Pin_20), U3.6 (-); no longer HEAD_L1.4 (Pin_4)
- net H_LED_OUT: now also HEAD_R1.19 (Pin_19); no longer HEAD_L1.7 (Pin_7)
- net S1: now also SOCK_L1.17 (Pin_17); no longer SOCK_L1.1 (Pin_1)
- net S2: now also SOCK_L1.18 (Pin_18); no longer SOCK_L1.2 (Pin_2)
- net S3: now also SOCK_L1.19 (Pin_19); no longer SOCK_L1.3 (Pin_3)
- net S4: now also SOCK_L1.20 (Pin_20); no longer SOCK_L1.4 (Pin_4)
- net S_3V3_A: now also SOCK_R1.17 (Pin_17); no longer SOCK_L1.8 (Pin_8)
- net S_GND: now also D1.1 (K), SOCK_R1.18 (Pin_18); no longer SOCK_L1.9 (Pin_9)
- net S_LED_OUT: now also SOCK_R1.19 (Pin_19); no longer SOCK_L1.7 (Pin_7)
- net +5V renamed H_+5V
- net -10V_REF renamed S_-10V_REF
- net S_-10V_REF: now also SOCK_R1.20 (Pin_20); no longer SOCK_L1.6 (Pin_6)
- net 3V3_A renamed H_3V3_A
- net H_3V3_A: now also HEAD_R1.17 (Pin_17), U3.8 (V+); no longer HEAD_L1.8 (Pin_8)
- net ADC_IN_0 renamed H_ADC_IN_0
- net H_ADC_IN_0: now also U3.1
- net ADC_IN_1 renamed H_ADC_IN_1
- net H_ADC_IN_1: now also U3.7
- net AUDIO_IN_L renamed H_AUDIO_IN_L
- net AUDIO_OUT_L renamed H_AUDIO_OUT_L
- net H5: no longer names the net of HEAD_L1.5 (Pin_5)
- net H5: no longer SEED1.12 (I2C1_SCL)
- net H6 renamed H_-10V_REF
- net H_-10V_REF: now also HEAD_R1.20 (Pin_20); no longer HEAD_L1.6 (Pin_6)
- net S5: no longer names the net of SOCK_L1.5 (Pin_5)
- net S5: no longer SW1.2 (B)
- new net: C12.2, C13.2, J4.10 (+12V), J4.9 (+12V), R19.1
- new net: C11.1, C14.1, J4.1 (-12V), J4.2 (-12V)
- new net H_SWITCH_IN: HEAD_R1.12 (Pin_12), SEED1.12 (I2C1_SCL)
- new net S_SWITCH_IN: SOCK_R1.12 (Pin_12), SW1.2 (B)
- no-connect marks 5 -> 97
Other:
- note added: "The seed is on the SOCKET board The pots/leds etc are on the HEADER board"
- moved on the sheet: C7, C8, D1, HEAD_L1, R19, R20, SEED1, SOCK_L1, U1
